File: teensy_board/sm_board.kicad_pcb (KiCad board)
At the start: 2 copper layers, 85.5 x 54.5 mm, 55 parts, among them IC1 DRV8833RTYT, J1 Conn_01x06, J10 Conn_01x03, J11 CONN_01X02, J13 Conn_01x02, J14 Conn_01x02, J2 Conn_01x06, J3 Conn_01x06, J4 Conn_01x03, J5 Conn_01x03, J6 Conn_01x03, J7 Conn_01x03, J8 Conn_01x03, J9 Conn_01x03, U1 Teensy3.6, U3 tps82130

Commit message: After review meeting
Parts:
- moved REF** 0.50 mm to (66.0, 102.5)
- moved REF** 0.27 mm to (123.5, 114.0)
Changed lines of the file:
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@@
     (links 136)
     (no_connects 3)
-    (area 62.399999 62.399999 147.955501 117.100001)
+    (area 56.942857 60.20374 147.955501 119.627973)
     (thickness 1.6)
     (drawings 6)
@@
   )
   (module Mounting_Holes:MountingHole_2.2mm_M2 (layer F.Cu)
-    (at 66.5 102.5)
+    (at 66 102.5)
     (descr "Mounting Hole 2.2mm, no annular, M2")
     (tags "mounting hole 2.2mm no annular m2")
@@
   )
   (module Mounting_Holes:MountingHole_2.2mm_M2 (layer F.Cu)
-    (at 123.25 113.9)
+    (at 123.5 114)
     (descr "Mounting Hole 2.2mm, no annular, M2")
     (tags "mounting hole 2.2mm no annular m2")
@@
   (gr_line (start 126.5 62.5) (end 62.5 62.5) (angle 90) (layer Edge.Cuts) (width 0.2))
   (gr_circle (center 146.685 104.10952) (end 147.955 104.10952) (layer Edge.Cuts) (width 0.001))
-  (segment (start 75.84576 100.38588) (end 76.74864 100.38588) (width 0.25) (layer F.Cu) (net 1) (status 400000))
+  (segment (start 75.84576 100.38588) (end 76.74864 100.38588) (width 0.25) (layer F.Cu) (net 1))
   (via (at 76.75372 100.39096) (size 0.6858) (drill 0.3302) (layers F.Cu B.Cu) (net 1))
   (segment (start 76.74864 100.38588) (end 76.75372 100.39096) (width 0.25) (layer F.Cu) (net 1))
-  (segment (start 121.59488 104.20594) (end 124.08154 104.20594) (width 0.25) (layer F.Cu) (net 1) (status C00000))
-  (segment (start 124.08154 104.20594) (end 124.16536 104.12212) (width 0.25) (layer F.Cu) (net 1) (status C00000))
-  (segment (start 114 104.3) (end 116.47162 104.3) (width 0.25) (layer F.Cu) (net 1) (status C00000))
-  (segment (start 116.47162 104.3) (end 116.5098 104.26182) (width 0.25) (layer F.Cu) (net 1) (status C00000))
-  (segment (start 111.43996 90.18524) (end 112.6236 90.18524) (width 0.25) (layer F.Cu) (net 1) (status 400000))
-  (segment (start 112.69472 103.28656) (end 111.68128 104.3) (width 0.25) (layer F.Cu) (net 1) (status 800000))
+  (segment (start 121.59488 104.20594) (end 124.08154 104.20594) (width 0.25) (layer F.Cu) (net 1))
+  (segment (start 124.08154 104.20594) (end 124.16536 104.12212) (width 0.25) (layer F.Cu) (net 1))
+  (segment (start 114 104.3) (end 116.47162 104.3) (width 0.25) (layer F.Cu) (net 1))
+  (segment (start 116.47162 104.3) (end 116.5098 104.26182) (width 0.25) (layer F.Cu) (net 1))
+  (segment (start 111.43996 90.18524) (end 112.6236 90.18524) (width 0.25) (layer F.Cu) (net 1))
+  (segment (start 112.69472 103.28656) (end 111.68128 104.3) (width 0.25) (layer F.Cu) (net 1))
   (segment (start 112.69472 101.98608) (end 112.69472 103.28656) (width 0.25) (layer F.Cu) (net 1))
   (via (at 112.69472 101.98608) (size 0.6858) (drill 0.3302) (layers F.Cu B.Cu) (net 1))
@@
   (segment (start 113.32464 90.88628) (end 113.32464 95.16364) (width 0.25) (layer F.Cu) (net 1))
   (segment (start 112.6236 90.18524) (end 113.32464 90.88628) (width 0.25) (layer F.Cu) (net 1))
-  (segment (start 111.68128 104.3) (end 111.4 104.3) (width 0.25) (layer F.Cu) (net 1) (status C00000))
+  (segment (start 111.68128 104.3) (end 111.4 104.3) (width 0.25) (layer F.Cu) (net 1))
   (segment (start 106.4 104.3) (end 108.9 104.3) (width 0.375) (layer F.Cu) (net 1))
   (segment (start 108.9 104.3) (end 111.4 104.3) (width 0.375) (layer F.Cu) (net 1))
@@
   (segment (start 81.45 102.45) (end 81.45 104.1) (width 0.375) (layer B.Cu) (net 3))
   (via (at 81.45 104.1) (size 0.6858) (drill 0.3302) (layers F.Cu B.Cu) (net 3))
-  (segment (start 110.84556 108.9762) (end 111.51252 108.9762) (width 0.25) (layer F.Cu) (net 3) (status 800000))
+  (segment (start 110.84556 108.9762) (end 111.51252 108.9762) (width 0.25) (layer F.Cu) (net 3))
   (segment (start 110.00232 109.81944) (end 110.84556 108.9762) (width 0.25) (layer F.Cu) (net 3))
   (segment (start 110.00232 110.7948) (end 110.00232 109.81944) (width 0.25) (layer F.Cu) (net 3))

Commit message: Boards that got ordered
Parts:
- removed REF** (x3): MountingHole_2.2mm_M2, Mounting_Holes:MountingHole_2.2mm_M2
Connections:
- net m1a renamed AOUT1
- net m1b renamed AOUT2
- net m2a renamed BOUT1
- net m2b renamed BOUT2
- net rx_imu renamed rx
- net tx_imu renamed tx
- J2 pad 1: Net-(J2-Pad1) -> (no net)
- J2 pad 5: Net-(J2-Pad5) -> (no net)
- U1 pad 11: MOSI -> CS0
- U1 pad 12: MISO -> CS1
- U1 pad 13: CS0 -> MOSI
- U1 pad 14: CS1 -> MISO
- U1 pad 16: Net-(U1-Pad16) -> (no net)
- U1 pad 25: Net-(U1-Pad25) -> (no net)
- U1 pad 28: Net-(U1-Pad28) -> (no net)
- U1 pad 38: Net-(U1-Pad38) -> (no net)
- U1 pad 4: ex_imu -> (no net)
- U1 pad 41: Net-(U1-Pad41) -> (no net)
- U1 pad 42: Net-(U1-Pad42) -> (no net)
- U1 pad 43: Net-(U1-Pad43) -> (no net)
- U1 pad 44: Net-(U1-Pad44) -> (no net)
- U1 pad 45: Net-(U1-Pad45) -> (no net)
- U1 pad 46: Net-(U1-Pad46) -> (no net)
- U1 pad 47: Net-(U1-Pad47) -> (no net)
- U1 pad 48: Net-(U1-Pad48) -> (no net)
- U1 pad 49: Net-(U1-Pad49) -> (no net)
- U1 pad 5: scl_imu -> (no net)
- U1 pad 51: Net-(U1-Pad51) -> (no net)
- U1 pad 6: sda_imu -> (no net)
- U3 pad 7: Net-(U3-Pad7) -> (no net)
- U3 pad 8: Net-(U3-Pad8) -> (no net)
Routing:
- net +3V3: track 100.2 -> 149.6 mm, vias 4 -> 6
- net CS1: track 17.3 -> 31.8 mm, vias 2 -> 3
- net CS0: track 14.9 -> 17.4 mm
- net MISO: track 29.9 -> 32.1 mm, vias 3 -> 4
- net MOSI: track 29.0 -> 29.9 mm, vias 2 -> 4
Other:
- outline, holes or cut-outs redrawn
