File: teensy_board/sm_board.sch (KiCad schematic (older format))
At the start: 45 parts, among them J0 CONN_01X03, J1 CONN_01X03, J10 CONN_01X04, J11 CONN_01X02, J12 CONN_02X04, J2 CONN_01X03, J3 CONN_01X03, J4 CONN_01X03, J5 CONN_01X03, J6 CONN_01X03, J7 CONN_01X02, J8 CONN_01X02, J9 CONN_01X04, U1 Teensy3.6, U2 drv8833, U3 tps82130

Commit message: I think im done the schematic for tonight
Parts:
- removed J0, J1, J2, J3, J4, J5, J6: CONN_01X03, Pin_Headers:Pin_Header_Straight_1x03_Pitch2.54mm, symbol CONN_01X03
- removed J10, J9: CONN_01X04, Pin_Headers:Pin_Header_Straight_1x04_Pitch2.54mm, symbol CONN_01X04
- removed J7, J8: CONN_01X02, Pin_Headers:Pin_Header_Straight_1x02_Pitch2.54mm, symbol CONN_01X02
- removed U2: drv8833, drv8833:drv8833, symbol drv8833
- added C10: 0.01uC, Capacitors_SMD:C_0603, symbol C
- added C11: 10uC, Capacitors_SMD:C_0603, symbol C
- added C9: 2.2uC, Capacitors_SMD:C_0603, symbol C
- added IC1: DRV8833RTYT, Housings_DFN_QFN:WQFN-16-1EP_4x4mm_Pitch0.65mm, symbol DRV8833RTYT
- added J1, J3: Conn_01x06, Connector_Molex:Molex_CLIK-Mate_502386-0670_1x06_P1.25mm_Horizontal, symbol Conn_01x06
- added J10, J4, J5, J6, J7, J8, J9: Conn_01x03, Connector_Molex:Molex_CLIK-Mate_502386-0370_1x03_P1.25mm_Horizontal, symbol Conn_01x03
- added J13, J14: Conn_01x02, Connector_Molex:Molex_CLIK-Mate_502494-0270_1x02_P2.00mm_Horizontal, symbol Conn_01x02
- added J2: Conn_01x06, Pin_Headers:Pin_Header_Straight_1x06_Pitch2.54mm, symbol Conn_01x06
- added R11, R2: R, Resistors_SMD:R_0603, symbol R
- C0, C1, C2, C3, C4, C5, C6, C7, C8: footprint Capacitors_SMD:C_0805 -> Capacitors_SMD:C_0603
- D0, D1, D2, D3, D4, D5, D6, D7: footprint LEDs:LED_0805 -> LEDs:LED_0603
- R0, R1, R10, R3, R4, R5, R6, R7, R8, R9: footprint Resistors_SMD:R_0805 -> Resistors_SMD:R_0603
- U1: footprint Teensy:Teensy35_36_custom -> Teensy:Teensy35_36
Connections:
- net +3V3: now also J1.5 (Pin_5), J3.5 (Pin_5)
- net +5V: now also C10.1, J10.2 (Pin_2), J2.4 (Pin_4), J4.2 (Pin_2), J5.2 (Pin_2), J6.2 (Pin_2), J7.2 (Pin_2), J8.2 (Pin_2), J9.2 (Pin_2)
- net GND: now also C11.2, C9.1, IC1.11 (GND_(PPAD)(1)), IC1.17 (GND_(PPAD)(2)), J1.6 (Pin_6), J2.6 (Pin_6), J3.6 (Pin_6), R11.2, R2.2
- net GNDA: now also J10.3 (Pin_3), J4.3 (Pin_3), J5.3 (Pin_3), J6.3 (Pin_3), J7.3 (Pin_3), J8.3 (Pin_3), J9.3 (Pin_3)
- net dist_a_0: now also J4.1 (Pin_1)
- net dist_a_1: now also J5.1 (Pin_1)
- net dist_a_2: now also J6.1 (Pin_1)
- net dist_a_3: now also J7.1 (Pin_1)
- net dist_a_4: now also J8.1 (Pin_1)
- net dist_a_5: now also J9.1 (Pin_1)
- net dist_a_6: now also J10.1 (Pin_1)
- net m_a1: now also IC1.14 (AIN1)
- net m_a2: now also IC1.13 (AIN2)
- net m_b1: now also IC1.7 (BIN1)
- net m_b2: now also IC1.8 (BIN2)
- net rx_imu: now also J2.3 (Pin_3)
- net tx_imu: now also J2.2 (Pin_2)
- net SCK: now reaches U1.40 (13_SCK0_LED)
- net SCK: now also J1.3 (Pin_3), J3.3 (Pin_3)
- net enc_a1 renamed MOSI
- net MOSI: now also J1.1 (Pin_1), J3.1 (Pin_1)
- net enc_a2 renamed MISO
- net MISO: now also J1.2 (Pin_2), J3.2 (Pin_2)
- net enc_b1 renamed cs0
- net enc_b2 renamed cs1
- new net: IC1.1 (AISEN), R2.1
- new net: C11.1, IC1.10 (VM)
- new net: C9.2, IC1.12 (VINT)
- new net: IC1.4 (BISEN), R11.1
- new net: C10.2, IC1.9 (VCP)
- new net CS0: J1.4 (Pin_4)
- new net CS1: J3.4 (Pin_4)
- new net m1a: IC1.16 (AOUT1), J13.1 (Pin_1)
- new net m1b: IC1.2 (AOUT2), J13.2 (Pin_2)
- new net m2a: IC1.5 (BOUT1), J14.1 (Pin_1)
- new net m2b: IC1.3 (BOUT2), J14.2 (Pin_2)
Other:
- moved on the sheet: C0, C1, J11, J12, R0, R1, S0, S1, U3

Commit message: I think this is done
Parts:
- added R12, R13: R, Resistors_SMD:R_0402, symbol R
- C0, C1, C10, C11, C2, C3, C4, C5, C6, C7, C8, C9: footprint Capacitors_SMD:C_0603 -> Capacitors_SMD:C_0402
- J10, J4, J5, J6, J7, J8, J9: footprint Connector_Molex:Molex_CLIK-Mate_502386-0370_1x03_P1.25mm_Horizontal -> Connector_Molex:Molex_CLIK-Mate_502382-0370_1x03_P1.25mm_Vertical
- R0, R1, R10, R11, R2, R3, R4, R5, R6, R7, R8, R9: footprint Resistors_SMD:R_0603 -> Resistors_SMD:R_0402
- U1: footprint Teensy:Teensy35_36 -> Teensy2:Teensy35_36_custom
Connections:
- net +3V3: now also C2.2, C3.2, C4.2, C5.2, C6.2, C7.2, C8.2, J10.2 (Pin_2), J4.2 (Pin_2), J5.2 (Pin_2), J6.2 (Pin_2), J7.2 (Pin_2), J8.2 (Pin_2), J9.2 (Pin_2)
- net +5V: no longer C2.2, C3.2, C4.2, C5.2, C6.2, C7.2, C8.2, J10.2 (Pin_2), J4.2 (Pin_2), J5.2 (Pin_2), J6.2 (Pin_2), J7.2 (Pin_2), J8.2 (Pin_2), J9.2 (Pin_2)
- net +BATT: now also R12.2
- net GND: now also R13.1
- net BattCheck: now reaches U1.37 (A21_DAC0)
- net BattCheck: now also R12.1, R13.2

Commit message: After review meeting
Parts:
- removed J12: CONN_02X04, Pin_Headers:Pin_Header_Straight_2x04_Pitch2.54mm, symbol CONN_02X04
Connections:
- net MISO: now also U1.14 (12_MISO0); no longer U1.12 (10_PWM_TX2_CS0)
- net MOSI: now also U1.13 (11_MOSI0); no longer U1.11 (9_PWM_RX2_CS0)
- net cs0: now also U1.11 (9_PWM_RX2_CS0); no longer U1.13 (11_MOSI0)
- net cs1: now also U1.12 (10_PWM_TX2_CS0); no longer U1.14 (12_MISO0)
- net m1a renamed AOUT1
- net m1b renamed AOUT2
- net m2a renamed BOUT1
- net m2b renamed BOUT2
- net rx_imu renamed rx
- net tx_imu renamed tx
Other:
- moved on the sheet: R12, R13
Changed lines of the file:
@@
 Wire Wire Line
 	3250 1800 3450 1800
-$Comp
-L CONN_02X04 J12
-U 1 1 58ECF8BE
-P 4400 850
-F 0 "J12" H 4400 1100 50  0000 C CNN
-F 1 "CONN_02X04" H 4400 600 50  0000 C CNN
-F 2 "Pin_Headers:Pin_Header_Straight_2x04_Pitch2.54mm" H 4400 -350 50  0001 C CNN
-F 3 "" H 4400 -350 50  0001 C CNN
-	1    4400 850
-	1    0    0    -1
-$EndComp
-Text GLabel 4000 700  0    60   Input ~ 0
-sda_imu
-Text GLabel 4000 800  0    60   Input ~ 0
-tx_imu
-Text GLabel 4800 700  2    60   Input ~ 0
-scl_imu
-Text GLabel 4800 800  2    60   Input ~ 0
-rx_imu
-Text GLabel 4800 1000 2    60   Input ~ 0
-ex_imu
-Wire Wire Line
-	4000 700  4150 700
-Wire Wire Line
-	4000 800  4150 800
-Wire Wire Line
-	4800 700  4650 700
-Wire Wire Line
-	4650 800  4800 800
-Wire Wire Line
-	4800 1000 4650 1000
-$Comp
-L GND #PWR025
-U 1 1 58ED2351
-P 4000 1000
-F 0 "#PWR025" H 4000 750 50  0001 C CNN
-F 1 "GND" H 4000 850 50  0000 C CNN
-F 2 "" H 4000 1000 50  0001 C CNN
-F 3 "" H 4000 1000 50  0001 C CNN
-	1    4000 1000
-	0    1    1    0
-$EndComp
-Wire Wire Line
-	4000 1000 4150 1000
-Wire Wire Line
-	4150 900  4100 900
-Wire Wire Line
-	4100 900  4100 1000
-Connection ~ 4100 1000
-$Comp
-L +3.3V #PWR026
-U 1 1 58ED3028
-P 5150 900
-F 0 "#PWR026" H 5150 750 50  0001 C CNN
-F 1 "+3.3V" H 5150 1040 50  0000 C CNN
-F 2 "" H 5150 900 50  0001 C CNN
-F 3 "" H 5150 900 50  0001 C CNN
-	1    5150 900
-	0    1    1    0
-$EndComp
-Wire Wire Line
-	4650 900  5150 900
 Text GLabel 1100 800  0    60   Input ~ 0
-tx_imu
+tx
 Text GLabel 1100 700  0    60   Input ~ 0
-rx_imu
+rx
 Wire Wire Line
 	1100 1200 1250 1200
@@
 Wire Wire Line
 	3250 3100 3450 3100
+Text GLabel 1100 1800 0    60   Input ~ 0
+MOSI
+Text GLabel 1100 1900 0    60   Input ~ 0
+MISO
 Text GLabel 1100 1600 0    60   Input ~ 0
-MOSI
+cs0
 Text GLabel 1100 1700 0    60   Input ~ 0
-MISO
-Text GLabel 1100 1800 0    60   Input ~ 0
-cs0
-Text GLabel 1100 1900 0    60   Input ~ 0
 cs1
 Wire Wire Line
@@
 $EndComp
 Text GLabel 2000 5400 1    60   Input ~ 0
-m1a
+AOUT1
 Text GLabel 1250 6600 0    60   Input ~ 0
-m1b
+AOUT2
 Text GLabel 1250 6700 0    60   Input ~ 0
-m2b
+BOUT2
 Text GLabel 1900 7500 3    60   Input ~ 0
-m2a
+BOUT1
 Wire Wire Line
 	2900 6700 3700 6700
@@
 $EndComp
 Text GLabel 4450 1550 3    60   Input ~ 0
-tx_imu
+tx
 Text GLabel 4550 1550 3    60   Input ~ 0
-rx_imu
+rx
 $Comp
 L +5V #PWR034
@@
 $EndComp
 Text GLabel 6350 2550 3    60   Input ~ 0
-m1a
+AOUT1
 Text GLabel 6450 2550 3    60   Input ~ 0
-m1b
+AOUT2
 Text GLabel 6750 2550 3    60   Input ~ 0
-m2a
+BOUT1
 Text GLabel 6850 2550 3    60   Input ~ 0
-m2b
+BOUT2
 $Comp
 L GND #PWR040
@@
 L R R12
 U 1 1 5AAC0D56
-P 6250 3750
-F 0 "R12" V 6330 3750 50  0000 C CNN
-F 1 "R" V 6250 3750 50  0000 C CNN
-F 2 "Resistors_SMD:R_0402" V 6180 3750 50  0001 C CNN
-F 3 "" H 6250 3750 50  0001 C CNN
-	1    6250 3750
+P 6300 4950
+F 0 "R12" V 6380 4950 50  0000 C CNN
+F 1 "R" V 6300 4950 50  0000 C CNN
+F 2 "Resistors_SMD:R_0402" V 6230 4950 50  0001 C CNN
+F 3 "" H 6300 4950 50  0001 C CNN
+	1    6300 4950
 	0    1    1    0
 $EndComp
@@
 L R R13
 U 1 1 5AAC0DE4
-P 6650 3750
-F 0 "R13" V 6730 3750 50  0000 C CNN
-F 1 "R" V 6650 3750 50  0000 C CNN
-F 2 "Resistors_SMD:R_0402" V 6580 3750 50  0001 C CNN
-F 3 "" H 6650 3750 50  0001 C CNN
-	1    6650 3750
-	0    1    1    0
-$EndComp
-Wire Wire Line
-	6400 3750 6500 3750
-Wire Wire Line
-	6450 3350 6450 3750
-Connection ~ 6450 3750
-Wire Wire Line
-	6800 3750 6950 3750
+P 6700 4950
+F 0 "R13" V 6780 4950 50  0000 C CNN
+F 1 "R" V 6700 4950 50  0000 C CNN
+F 2 "Resistors_SMD:R_0402" V 6630 4950 50  0001 C CNN
+F 3 "" H 6700 4950 50  0001 C CNN
+	1    6700 4950
+	0    1    1    0
+$EndComp
+Wire Wire Line
+	6450 4950 6550 4950
+Wire Wire Line
+	6500 4550 6500 4950
+Connection ~ 6500 4950
+Wire Wire Line
+	6850 4950 7000 4950
 $Comp
 L GND #PWR041
 U 1 1 5AAC11C8
-P 6950 3750
-F 0 "#PWR041" H 6950 3500 50  0001 C CNN
-F 1 "GND" H 6950 3600 50  0000 C CNN
-F 2 "" H 6950 3750 50  0001 C CNN
-F 3 "" H 6950 3750 50  0001 C CNN
-	1    6950 3750
+P 7000 4950
+F 0 "#PWR041" H 7000 4700 50  0001 C CNN
+F 1 "GND" H 7000 4800 50  0000 C CNN
+F 2 "" H 7000 4950 50  0001 C CNN
+F 3 "" H 7000 4950 50  0001 C CNN
+	1    7000 4950
 	0    -1   -1   0
 $EndComp
@@
 L +BATT #PWR042
 U 1 1 5AAC127B
-P 6100 3750
-F 0 "#PWR042" H 6100 3600 50  0001 C CNN
-F 1 "+BATT" H 6100 3890 50  0000 C CNN
-F 2 "" H 6100 3750 50  0001 C CNN
-F 3 "" H 6100 3750 50  0001 C CNN
-	1    6100 3750
+P 6150 4950
+F 0 "#PWR042" H 6150 4800 50  0001 C CNN
+F 1 "+BATT" H 6150 5090 50  0000 C CNN
+F 2 "" H 6150 4950 50  0001 C CNN
+F 3 "" H 6150 4950 50  0001 C CNN
+	1    6150 4950
 	0    -1   -1   0
 $EndComp
 Text GLabel 1250 4200 0    60   Input ~ 0
 BattCheck
-Text GLabel 6450 3350 1    60   Input ~ 0
+Text GLabel 6500 4550 1    60   Input ~ 0
 BattCheck
 $Comp
